File: hardware/kicad/placa/placa.kicad_sch (KiCad schematic)
At the start: 49 parts, among them J1 USB-TYPE-C-008, J2 Bateria, J3 OLED SSD1306, J4 TTP223, J5 UART, J6 ULTRASONIDO, Q1 AO3400A, SW1 SW_SPST, SW2 SW_SPST, SW3 SW_SPST, U1 TP4056, U2 MT3608, U3 AMS1117, U4 ESP32-C3FH4, U5 TC4427xOA, X1 40MHz, 15pF

Commit message: n
Parts:
- removed R4: 3.3kΩ, PCM_JLCPCB:R_0402, symbol PCM_JLCPCB-Resistors:0402,3.3kΩ
- removed R5: 10kΩ, PCM_JLCPCB:R_0402, symbol PCM_JLCPCB-Resistors:0402,10kΩ
- removed TH2: Thermistor_NTC_US, symbol Device:Thermistor_NTC_US
- J2, J6: footprint (none) -> Library-Humi:PH2.0-2P
- J3: footprint (none) -> Connector_PinSocket_2.54mm:PinSocket_1x04_P2.54mm_Vertical
- J4, J5: footprint (none) -> Library-Humi:PH2.0-3P
- L1: footprint (none) -> Library-Humi:IND-10u-C2849472
- L2: footprint (none) -> Library-Humi:Ind-220u-C167899
- SW1: renamed from SW3; footprint (none) -> Library-Humi:PH2.0-2P
- SW2: renamed from SW1; footprint (none) -> Library-Humi:Pulsador-SMD_KMR2XXGXXX
- SW3: renamed from SW2; footprint (none) -> Library-Humi:Pulsador-SMD_KMR2XXGXXX
- renumbered R12 to R10, R6 to R4, R7 to R5, R8 to R6, R9 to R7, R10 to R8, R11 to R9
Connections:
- net TEMP is gone; now on net GND: U1.1 (TEMP)
Other:
- moved on the sheet: C2, D1, D2, R1, R2, R3, U1
